File: kicad/industrial_usb_hub/industrial_usb_hub.kicad_pcb (KiCad board)
At the start: 4 copper layers, 0 parts

Commit message: moved on to pcb editor, chose component placements, groups, now needs routing, and bro routing superspeed just sucks
Parts:
- added C1: 0.1µ, Capacitor_SMD:C_0201_0603Metric, F.Cu at (136.2, 97.5)
- added C10: 0.1µ, Capacitor_SMD:C_0201_0603Metric, F.Cu at (137.7, 97.5)
- added C11: 0.1µ, Capacitor_SMD:C_0201_0603Metric, F.Cu at (137.7, 96.8)
- added C12: 0.1µ, Capacitor_SMD:C_0201_0603Metric, F.Cu at (137.7, 96.0)
- added C13: 0.1µ, Capacitor_SMD:C_0201_0603Metric, F.Cu at (130.0, 110.8)
- added C14: 0.1µ, Capacitor_SMD:C_0201_0603Metric, F.Cu at (131.0, 110.7)
- added C15: 0.1µ, Capacitor_SMD:C_0201_0603Metric, F.Cu at (136.8, 122.0)
- added C16: 0.1µ, Capacitor_SMD:C_0201_0603Metric, F.Cu at (127.8, 112.8)
- added C17: 0.1µ, Capacitor_SMD:C_0201_0603Metric, F.Cu at (141.8, 105.0)
- added C18: 0.1µ, Capacitor_SMD:C_0201_0603Metric, F.Cu at (141.8, 104.2)
- added C19: 0.1µ, Capacitor_SMD:C_0201_0603Metric, F.Cu at (140.2, 102.0)
- added C2: 0.1µ, Capacitor_SMD:C_0201_0603Metric, F.Cu at (137.7, 99.8)
- added C20: 10µ, Capacitor_SMD:C_0201_0603Metric, F.Cu at (144.8, 103.3)
- added C21: 10µ, Capacitor_SMD:C_0201_0603Metric, F.Cu at (127.2, 104.1)
- added C22: 0.1µ, Capacitor_SMD:C_0201_0603Metric, F.Cu at (129.4, 121.7)
- added C23: 33p, Capacitor_SMD:C_0201_0603Metric, F.Cu at (139.0, 111.0)
- added C24: 33p, Capacitor_SMD:C_0201_0603Metric, F.Cu at (132.8, 111.2)
- added C25: 0.1µ, Capacitor_SMD:C_0201_0603Metric, F.Cu at (141.0, 99.5)
- added C26: 0.1µ, Capacitor_SMD:C_0201_0603Metric, F.Cu at (141.0, 98.5)
- added C27: 0.1µ, Capacitor_SMD:C_0201_0603Metric, F.Cu at (135.0, 97.9)
- added C28: 0.1µ, Capacitor_SMD:C_0201_0603Metric, F.Cu at (133.5, 97.9)
- added C29: 0.1µ, Capacitor_SMD:C_0201_0603Metric, F.Cu at (130.8, 99.2)
- added C3: 0.1µ, Capacitor_SMD:C_0201_0603Metric, F.Cu at (136.2, 98.2)
- added C30: 0.1µ, Capacitor_SMD:C_0201_0603Metric, F.Cu at (130.8, 100.2)
- added C31: 0.1µ, Capacitor_SMD:C_0201_0603Metric, F.Cu at (137.5, 85.5)
- added C32: 10µ, Capacitor_SMD:C_0201_0603Metric, F.Cu at (141.8, 86.5)
- added C33: 0.1µ, Capacitor_SMD:C_0201_0603Metric, F.Cu at (125.2, 103.5)
- added C34: 10µ, Capacitor_SMD:C_0201_0603Metric, F.Cu at (122.2, 104.6)
- added C35: 0.1µ, Capacitor_SMD:C_0201_0603Metric, F.Cu at (127.2, 85.5)
- added C36: 10µ, Capacitor_SMD:C_0201_0603Metric, F.Cu at (123.2, 84.8)
- added C37: 10µ, Capacitor_SMD:C_0201_0603Metric, F.Cu at (128.2, 110.3)
- added C38: 22µ, Capacitor_SMD:C_0201_0603Metric, F.Cu at (134.4, 73.2)
- added C39: 6.8n, Capacitor_SMD:C_0201_0603Metric, F.Cu at (129.4, 73.3)
- added C4: 0.1µ, Capacitor_SMD:C_0201_0603Metric, F.Cu at (136.2, 99.0)
- added C40: 1µ, Capacitor_SMD:C_0201_0603Metric, F.Cu at (131.5, 71.0)
- added C41: 44µ, Capacitor_SMD:C_0201_0603Metric, F.Cu at (129.0, 74.5)
- added C42: 22µ, Capacitor_SMD:C_0201_0603Metric, F.Cu at (140.5, 74.2)
- added C43: 6.8n, Capacitor_SMD:C_0201_0603Metric, F.Cu at (135.8, 74.2)
- added C44: 1µ, Capacitor_SMD:C_0201_0603Metric, F.Cu at (140.5, 73.5)
- added C45: 44µ, Capacitor_SMD:C_0201_0603Metric, F.Cu at (135.0, 75.0)
- added C5: 0.1µ, Capacitor_SMD:C_0201_0603Metric, F.Cu at (136.2, 99.8)
- added C6: 0.1µ, Capacitor_SMD:C_0201_0603Metric, F.Cu at (137.7, 95.2)
- added C7: 0.1µ, Capacitor_SMD:C_0201_0603Metric, F.Cu at (137.7, 94.5)
- added C8: 0.1µ, Capacitor_SMD:C_0201_0603Metric, F.Cu at (137.7, 99.0)
- added C9: 0.1µ, Capacitor_SMD:C_0201_0603Metric, F.Cu at (137.7, 98.2)
- added J1: USB3_A, Connector_USB:USB3_A_Molex_48393-001, F.Cu at (150.6, 80.8)
- added J2: USB_C_Receptacle, personal_library:BELFUSE_SS-52400-003, F.Cu at (133.3, 130.0)
- added J3: USB3_A, Connector_USB:USB3_A_Molex_48393-001, F.Cu at (117.4, 96.8)
- added J4: USB3_A, Connector_USB:USB3_A_Molex_48393-001, F.Cu at (117.5, 73.8)
- added J6: USB3_A, Connector_USB:USB3_A_Molex_48393-001, F.Cu at (150.6, 103.8)
- added L1: 1.5µ, Inductor_SMD:L_Taiyo-Yuden_NR-40xx, F.Cu at (131.0, 78.5)
- added L2: 1.5µ, Inductor_SMD:L_Taiyo-Yuden_NR-40xx, F.Cu at (138.0, 78.5)
- added R1: 887, Resistor_SMD:R_0201_0603Metric, F.Cu at (134.0, 121.0)
- added R10: 10k, Resistor_SMD:R_0201_0603Metric, F.Cu at (129.5, 109.2)
- added R11: 10, Resistor_SMD:R_0201_0603Metric, F.Cu at (128.5, 107.2)
- added R12: 200k, Resistor_SMD:R_0201_0603Metric, F.Cu at (128.5, 108.0)
- added R13: 10k, Resistor_SMD:R_0201_0603Metric, F.Cu at (128.5, 106.5)
- added R14: 10k, Resistor_SMD:R_0201_0603Metric, F.Cu at (128.5, 105.8)
- added R15: 20, Resistor_SMD:R_0201_0603Metric, F.Cu at (129.7, 71.7)
- added R16: 30k, Resistor_SMD:R_0201_0603Metric, F.Cu at (131.2, 75.2)
- added R17: 40.2k, Resistor_SMD:R_0201_0603Metric, F.Cu at (129.0, 75.2)
- added R18: 13k, Resistor_SMD:R_0201_0603Metric, F.Cu at (130.2, 75.2)
- added R19: 20, Resistor_SMD:R_0201_0603Metric, F.Cu at (140.5, 72.5)
- added R2: 5.6k, Resistor_SMD:R_0201_0603Metric, F.Cu at (144.8, 101.5)
- added R20: 75k, Resistor_SMD:R_0201_0603Metric, F.Cu at (137.4, 75.8)
- added R21: 40.2k, Resistor_SMD:R_0201_0603Metric, F.Cu at (135.0, 75.8)
- added R22: 82k, Resistor_SMD:R_0201_0603Metric, F.Cu at (136.2, 75.5)
- added R23: 100k, Resistor_SMD:R_0201_0603Metric, F.Cu at (133.2, 73.6)
- added R24: 10k, Resistor_SMD:R_0201_0603Metric, F.Cu at (139.2, 113.5)
- added R3: 43k, Resistor_SMD:R_0201_0603Metric, F.Cu at (127.9, 104.5)
- added R4: 49.9k, Resistor_SMD:R_0201_0603Metric, F.Cu at (126.8, 105.2)
- added R5: 887, Resistor_SMD:R_0201_0603Metric, F.Cu at (129.4, 122.4)
- added R6: 12k, Resistor_SMD:R_0201_0603Metric, F.Cu at (138.5, 108.2)
- added R7: 5.6k, Resistor_SMD:R_0201_0603Metric, F.Cu at (141.8, 85.1)
- added R8: 5.6k, Resistor_SMD:R_0201_0603Metric, F.Cu at (122.2, 106.1)
- added R9: 5.6k, Resistor_SMD:R_0201_0603Metric, F.Cu at (123.2, 86.2)
- added U1: USB5744-I_2G, personal_library:USB5744-QFN40P700X700X100-57N, F.Cu at (133.6, 104.8)
- added U2: HD3SS3212IRKSR, personal_library:QFN50P450X250X100-21N, B.Cu at (132.8, 117.8)
- added U3: TUSB321, Package_DFN_QFN:Texas_X2QFN-12_1.6x1.6mm_P0.4mm, F.Cu at (139.6, 115.4)
- added U4: SY6280, personal_library:SOT23-5, F.Cu at (142.2, 102.0)
- added U5: SY6280, personal_library:SOT23-5, F.Cu at (139.2, 85.5)
- added U6: SY6280, personal_library:SOT23-5, F.Cu at (124.8, 105.2)
- added U7: SY6280, personal_library:SOT23-5, F.Cu at (125.8, 85.5)
- added U8: MP2393GTL-P, MP2393GTL-P:SOT583_MP2393, F.Cu at (131.5, 73.0)
- added U9: MP2393GTL-P, MP2393GTL-P:SOT583_MP2393, F.Cu at (138.0, 74.0)
- added Y1: Crystal_GND24, personal_library:403I35D25M00000, F.Cu at (135.8, 111.2)
Routing:
- net /Upstream/TX1_N: track 0.00 -> 3.89 mm, vias 0 -> 1
- net /Upstream/TX1_P: track 0.00 -> 3.89 mm, vias 0 -> 1
- added copper zone on In1.Cu, net GND
Other:
- board outline added: 55.5 x 64 mm
